File: plate/fr4/bakeneko-60-fr4-split-spacebar-plate.kicad_pcb (KiCad board)
At the start: 2 copper layers, 285.8 x 95.2 mm, 0 parts

Commit message: Add some funny text
Other:
- board text added: "This Is Not A Plate"
- board text added: "Unbakeneko v0.1"
Changed lines of the file:
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@@
   (gr_arc (start 169.767499 73.230001) (mid 169.913946 72.876448) (end 170.267499 72.730001) (layer "Edge.Cuts") (width 0.2))
   (gr_arc (start 188.529999 105.280001) (mid 188.383552 105.633554) (end 188.029999 105.780001) (layer "Edge.Cuts") (width 0.2))
+  (gr_text "This Is Not A Plate" (at 138.8 88.31) (layer "F.SilkS")
+    (effects (font (size 1 1) (thickness 0.15)))
+  )
+  (gr_text "Unbakeneko v0.1" (at 138.51 71.28) (layer "F.SilkS")
+    (effects (font (size 1 1) (thickness 0.15)))
+  )
   (via (at 268.355499 80.280001) (size 0.8) (drill 0.4) (layers "F.Cu" "B.Cu") (net 0))
 )

Commit message: Add production zip for plate
Other:
- rule pad_to_mask_clearance: 0.051 -> 0
Changed lines of the file:
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@@
   )
   (setup
-    (pad_to_mask_clearance 0.051)
-    (solder_mask_min_width 0.25)
+    (stackup
+      (layer "F.SilkS" (type "Top Silk Screen"))
+      (layer "F.Paste" (type "Top Solder Paste"))
+      (layer "F.Mask" (type "Top Solder Mask") (thickness 0.01))
+      (layer "F.Cu" (type "copper") (thickness 0.035))
+      (layer "dielectric 1" (type "core") (thickness 1.51) (material "FR4") (epsilon_r 4.5) (loss_tangent 0.02))
+      (layer "B.Cu" (type "copper") (thickness 0.035))
+      (layer "B.Mask" (type "Bottom Solder Mask") (thickness 0.01))
+      (layer "B.Paste" (type "Bottom Solder Paste"))
+      (layer "B.SilkS" (type "Bottom Silk Screen"))
+      (copper_finish "None")
+      (dielectric_constraints no)
+    )
+    (pad_to_mask_clearance 0)
     (pcbplotparams
       (layerselection 0x00010fc_ffffffff)
@@
     (effects (font (size 1 1) (thickness 0.15)))
   )
-  (via (at 268.355499 80.280001) (size 0.8) (drill 0.4) (layers "F.Cu" "B.Cu") (net 0))
+  (via (at 138.8 88.42) (size 0.8) (drill 0.4) (layers "F.Cu" "B.Cu") (net 0))
 )
